Commit message: remove gripper from urdf

File: src/ur10_robot_description/urdf/ur10_without_gripper.xacro (robot description, xacro)
@@ -1,6 +1,6 @@
 <?xml version="1.0"?>
-<robot name="ur5" xmlns:xacro="http://www.ros.org/wiki/xacro">
-  <xacro:include filename="$(find ur5_robot_description)/urdf/ur5_joint_limited_robot.urdf.xacro" />
-  <xacro:include filename="$(find ur5_robot_description)/urdf/robotiq/robotiq_85_gripper.urdf.xacro" />
+<robot name="ur10" xmlns:xacro="http://www.ros.org/wiki/xacro">
+  <xacro:include filename="$(find ur10_robot_description)/urdf/ur5_joint_limited_robot.urdf.xacro" />
+  <xacro:include filename="$(find ur10_robot_description)/urdf/robotiq/robotiq_85_gripper.urdf.xacro" />
   <!-- Let's try convert this ur5 urdf to ur10 (2025.04.11) -->
   <!-- Robotiq Coupler -->
@@ -10,10 +10,10 @@
     <visual>
       <geometry>
-        <mesh filename="package://ur5_robot_description/meshes/coupler.stl" />
+        <mesh filename="package://ur10_robot_description/meshes/coupler.stl" />
       </geometry>
     </visual>
     <collision>
       <geometry>
-        <mesh filename="package://ur5_robot_description/meshes/coupler.stl" />
+        <mesh filename="package://ur10_robot_description/meshes/coupler.stl" />
       </geometry>
     </collision>

File: src/ur10_robot_description/urdf/ur5_robotiq85_gripper.xacro (robot description, xacro)
@@ -3,5 +3,4 @@
   <xacro:include filename="$(find ur5_robot_description)/urdf/ur5_joint_limited_robot.urdf.xacro" />
   <xacro:include filename="$(find ur5_robot_description)/urdf/robotiq/robotiq_85_gripper.urdf.xacro" />
-  <!-- Let's try convert this ur5 urdf to ur10 (2025.04.11) -->
   <!-- Robotiq Coupler -->
   <!--  + Height added by the coupler: 8mm -->
@@ -42,6 +41,6 @@
   <!-- </joint> -->
   <!-- Attach the robotiq 85 gripper -->
-  <!-- <xacro:robotiq_85_gripper prefix="" parent="robotiq_coupler" >
+  <xacro:robotiq_85_gripper prefix="" parent="robotiq_coupler" >
     <origin xyz="0 0 0.004" rpy="0 ${-pi/2} ${pi}"/>
-  </xacro:robotiq_85_gripper>  -->
+  </xacro:robotiq_85_gripper>
 </robot>
