Commit message: ur_description pa package from /opt/ros/humble/share and trying move view_ur.launch.py

File: src/nrs_path2/urdf/inc/ur10e_macro.xacro (robot description, xacro)
@@ -1,43 +1,27 @@
 <?xml version="1.0"?>
-<robot xmlns:xacro="http://wiki.ros.org/xacro">
-  <!--
-    Convenience wrapper for the 'ur_robot' macro which provides default values
-    for the various "parameters files" parameters for a UR10.
-    This file can be used when composing a more complex scene with one or more
-    UR10 robots.
-    While the generic 'ur_robot' macro could also be used, it would require
-    the user to provide values for all parameters, as that macro does not set
-    any model-specific defaults (not even for the generic parameters, such as
-    the visual and physical parameters and joint limits).
-    Refer to the main 'ur_macro.xacro' in this package for information about
-    use, contributors and limitations.
-    NOTE: users will most likely want to override *at least* the
-          'kinematics_parameters_file' parameter. Otherwise, a default kinematic
-          model will be used, which will almost certainly not correspond to any
-          real robot.
-  -->
-  <xacro:macro name="ur10e_robot" params="
-   prefix
-   joint_limits_parameters_file:='$(find nrs_path)/config/joint_limits.yaml'
-   kinematics_parameters_file:='$(find nrs_path)/config/default_kinematics.yaml'
-   physical_parameters_file:='$(find nrs_path)/config/physical_parameters.yaml'
-   visual_parameters_file:='$(find nrs_path)/config/visual_parameters.yaml'
-   transmission_hw_interface:=hardware_interface/PositionJointInterface
-   safety_limits:=false
-   safety_pos_margin:=0.15
-   safety_k_position:=20"
-  >
-    <xacro:include filename="$(find nrs_path)/urdf/inc/ur_macro.xacro"/>
-    <xacro:ur_robot
-      prefix="${prefix}"
-      joint_limits_parameters_file="${joint_limits_parameters_file}"
-      kinematics_parameters_file="${kinematics_parameters_file}"
-      physical_parameters_file="${physical_parameters_file}"
-      visual_parameters_file="${visual_parameters_file}"
-      transmission_hw_interface="${transmission_hw_interface}"
-      safety_limits="${safety_limits}"
-      safety_pos_margin="${safety_pos_margin}"
-      safety_k_position="${safety_k_position}"
-    />
-  </xacro:macro>
+<robot xmlns:xacro="http://ros.org/wiki/xacro">
+  <!-- ROS 2용 UR10e macro wrapper -->
+  <!-- 인자 선언 -->
+  <xacro:arg name="prefix" default=""/>
+  <xacro:arg name="joint_limits_parameters_file" default="package://nrs_path2/config/joint_limits.yaml"/>
+  <xacro:arg name="kinematics_parameters_file" default="package://nrs_path2/config/default_kinematics.yaml"/>
+  <xacro:arg name="physical_parameters_file" default="package://nrs_path2/config/physical_parameters.yaml"/>
+  <xacro:arg name="visual_parameters_file" default="package://nrs_path2/config/visual_parameters.yaml"/>
+  <xacro:arg name="transmission_hw_interface" default="hardware_interface/PositionJointInterface"/>
+  <xacro:arg name="safety_limits" default="false"/>
+  <xacro:arg name="safety_pos_margin" default="0.15"/>
+  <xacro:arg name="safety_k_position" default="20"/>
+  <!-- macro 정의된 파일 포함 -->
+  <xacro:include filename="package://nrs_path2/urdf/inc/ur_macro.xacro"/>
+  <!-- 매크로 호출 -->
+  <xacro:ur_robot
+    prefix="${prefix}"
+    joint_limits_parameters_file="${joint_limits_parameters_file}"
+    kinematics_parameters_file="${kinematics_parameters_file}"
+    physical_parameters_file="${physical_parameters_file}"
+    visual_parameters_file="${visual_parameters_file}"
+    transmission_hw_interface="${transmission_hw_interface}"
+    safety_limits="${safety_limits}"
+    safety_pos_margin="${safety_pos_margin}"
+    safety_k_position="${safety_k_position}" />
 </robot>

File: src/nrs_path2/urdf/inc/ur_macro.xacro (robot description, xacro)
@@ -42,6 +42,6 @@
      - Muhammad Asif Rana
   -->
-  <xacro:include filename="$(find nrs_path)/urdf/inc/ur_transmissions.xacro" />
-  <xacro:include filename="$(find nrs_path)/urdf/inc/ur_common.xacro" />
+  <xacro:include filename="$(find nrs_path2)/urdf/inc/ur_transmissions.xacro" />
+  <xacro:include filename="$(find nrs_path2)/urdf/inc/ur_common.xacro" />
   <xacro:macro name="ur_robot" params="
     prefix

File: src/nrs_path2/urdf/testbed.xacro (robot description, xacro)
@@ -2,5 +2,5 @@
 <robot name="ur10e_robot" xmlns:xacro="http://www.ros.org/wiki/xacro">
   <!-- Include the UR10 robot description -->
-  <xacro:include filename="$(find nrs_path)/urdf/ur10e.xacro" />
+  <xacro:include filename="$(find nrs_path2)/urdf/ur10e.xacro" />
   <!-- Define the testbed link -->
   <link name="testbed">
@@ -32,5 +32,5 @@
     <visual>
       <geometry>
-        <mesh filename="package://nrs_path/mesh/UR10e_roboworld_tooltip_m.stl" />
+        <mesh filename="package://nrs_path2/mesh/UR10e_roboworld_tooltip_m.stl" />
       </geometry>
       <material name="tooltip_gray">
@@ -40,5 +40,5 @@
     <collision>
       <geometry>
-        <mesh filename="package://nrs_path/mesh/UR10e_roboworld_tooltip_m.stl" />
+        <mesh filename="package://nrs_path2/mesh/UR10e_roboworld_tooltip_m.stl" />
       </geometry>
       <material name="tooltip_gray">
@@ -50,5 +50,5 @@
     <visual>
       <geometry>
-        <mesh filename="package://nrs_path/mesh/workpiece.stl" />
+        <mesh filename="package://nrs_path2/mesh/workpiece.stl" />
       </geometry>
       <material name="light_blue">
@@ -58,5 +58,5 @@
     <!-- <collision>
       <geometry>
-        <mesh filename="package://nrs_path/mesh/fenda_wrap.stl" />
+        <mesh filename="package://nrs_path2/mesh/fenda_wrap.stl" />
       </geometry>
       <material name="light_blue">

File: src/nrs_path2/urdf/ur.xacro (robot description, xacro)
@@ -2,5 +2,5 @@
 <robot xmlns:xacro="http://wiki.ros.org/xacro" name="$(arg robot_model)_robot">
    <!-- import main macro -->
-   <xacro:include filename="$(find nrs_path)/urdf/inc/ur_macro.xacro"/>
+   <xacro:include filename="$(find nrs_path2)/urdf/inc/ur_macro.xacro"/>
    <!-- parameters -->
    <xacro:arg name="joint_limit_params" default=""/>

File: src/nrs_path2/urdf/ur10e.xacro (robot description, xacro)
@@ -1,18 +1,13 @@
 <?xml version="1.0"?>
-<robot xmlns:xacro="http://wiki.ros.org/xacro" name="ur10e_robot">
-  <!--
-    This is a convenience top-level xacro which loads the macro for the UR10
-    which defines the default values for the various "parameters files"
-    parameters for a UR10.
-    This file is only useful when loading a stand-alone, completely isolated
-    robot with only default values for all parameters such as the kinematics,
-    visual and physical parameters and joint limits.
-    This file is not intended to be integrated into a larger scene or other
-    composite xacro.
-    Instead, xacro:include 'inc/ur10_macro.xacro' and override the defaults
-    for the arguments to that macro.
-    Refer to 'inc/ur_macro.xacro' for more information.
-  -->
-  <xacro:include filename="$(find nrs_path)/urdf/inc/ur10e_macro.xacro"/>
-  <xacro:ur10e_robot prefix="" />
+<robot xmlns:xacro="http://ros.org/wiki/xacro">
+  <!-- declare args for ROS 2 -->
+  <xacro:arg name="prefix" default=""/>
+  <xacro:arg name="safety_limits" default="false"/>
+  <xacro:arg name="safety_pos_margin" default="0.15"/>
+  <xacro:arg name="safety_k_position" default="20"/>
+  <xacro:ur10e_robot
+    prefix="${prefix}"
+    safety_limits="${safety_limits}"
+    safety_pos_margin="${safety_pos_margin}"
+    safety_k_position="${safety_k_position}" />
 </robot>
